File: pcb.kicad_pcb (KiCad board)
At the start: 4 copper layers, 103 x 56 mm, 34 parts, among them J3 USB_C_Receptacle_USB2.0_16P, Q1 2N3904, SW1 RESET, SW2 KEY IP5306, SW5 BOOT, U1 USBLC6-2SC6, U2 IP5306, U4 TLV75533PDBV, U6 ESP32-S3-WROOM-1

Commit message: Updated PCB fixed USB C facing inwards the board
Parts:
- moved J3 1.19 mm to (84.8, 59.0), turned to -90 degrees
Routing:
- net VBUS: track 59.9 -> 30.5 mm
- net GND: track 19.9 -> 13.9 mm, vias 5 -> 6
- net Net-(J3-CC2): track 13.0 -> 18.6 mm
- net Net-(J3-CC1): track 13.3 -> 18.6 mm
- net USB_D-: track 60.4 -> 56.3 mm
- net USB_D+: track 59.9 -> 56.0 mm
